File: tangnano9k_motordriver.kicad_sch (KiCad schematic)
At the start: 29 parts, among them J1 Jack-DC, J2 Screw_Terminal_01x04, J3 Screw_Terminal_01x04, J4 Reserve, J5 Reserve, J6 Reserve, J7 Reserve_PinHeader, SW1 RotaryEncoder, SW2 RotaryEncoder, SW3 SW_DIP_x08, U1 BP5293-5, U2 TB67S101ANG, U3 TangNano9K, U4 OSL641505-BB, U5 TB67S101ANG

Commit message: 3
Other:
- title: (none) -> MoterDriverBoard for Tang Nano 9K
Changed lines of the file:
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@@
 (kicad_sch (version 20211123) (generator eeschema)
   (paper "A4")
+  (title_block
+    (title "MoterDriverBoard for Tang Nano 9K")
+  )
   (junction (at 35.56 151.13) (diameter 0) (color 0 0 0 0)
   )

Commit message: 4
Parts:
- J1: footprint (none) -> Connector_BarrelJack:BarrelJack_Horizontal
- J7: footprint digikey-footprints:PinHeader_1x4_P2mm_Drill1mm -> Connector_PinHeader_2.54mm:PinHeader_1x04_P2.54mm_Vertical
- SW1, SW2: footprint (none) -> Rotary_Encoder:RotaryEncoder_Alps_EC11E-Switch_Vertical_H20mm
- SW3: footprint (none) -> Button_Switch_SMD:SW_DIP_SPSTx03_Slide_9.78x9.8mm_W8.61mm_P2.54mm
- TP1, TP2: footprint (none) -> TestPoint:TestPoint_Pad_D2.0mm
Changed lines of the file:
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@@
     (property "Reference" "SW3" (id 0) (at 237.49 41.91 0))
     (property "Value" "SW_DIP_x08" (id 1) (at 237.49 44.45 0))
-    (property "Footprint" "" (id 2) (at 237.49 59.69 0)
+    (property "Footprint" "Button_Switch_SMD:SW_DIP_SPSTx03_Slide_9.78x9.8mm_W8.61mm_P2.54mm" (id 2) (at 237.49 59.69 0)
       (effects (font (size 1.27 1.27)) hide)
     )
@@
       (effects (font (size 1.27 1.27)) (justify left))
     )
-    (property "Footprint" "" (id 2) (at 194.31 123.19 0)
+    (property "Footprint" "TestPoint:TestPoint_Pad_D2.0mm" (id 2) (at 194.31 123.19 0)
       (effects (font (size 1.27 1.27)) hide)
     )
@@
     )
     (property "Value" "RotaryEncoder" (id 1) (at 138.43 85.09 0))
-    (property "Footprint" "" (id 2) (at 142.24 88.646 0)
+    (property "Footprint" "Rotary_Encoder:RotaryEncoder_Alps_EC11E-Switch_Vertical_H20mm" (id 2) (at 142.24 88.646 0)
       (effects (font (size 1.27 1.27)) hide)
     )
@@
       (effects (font (size 1.27 1.27)) (justify left))
     )
-    (property "Footprint" "" (id 2) (at 222.25 45.72 0)
+    (property "Footprint" "TestPoint:TestPoint_Pad_D2.0mm" (id 2) (at 222.25 45.72 0)
       (effects (font (size 1.27 1.27)) hide)
     )
@@
       (effects (font (size 1.27 1.27)) (justify right))
     )
-    (property "Footprint" "" (id 2) (at 44.45 22.606 0)
+    (property "Footprint" "Connector_BarrelJack:BarrelJack_Horizontal" (id 2) (at 44.45 22.606 0)
       (effects (font (size 1.27 1.27)) hide)
     )
@@
     (pin "4")
   )
-  (symbol (lib_id "455-1706-nd:455-1706-ND") (at 229.87 114.3 90) (unit 1)
-    (in_bom yes) (on_board yes) (fields_autoplaced)
-    (property "Reference" "J7" (id 0) (at 233.68 109.2199 90)
+  (symbol (lib_name "455-1706-ND_1") (lib_id "455-1706-nd:455-1706-ND") (at 229.87 114.3 90) (unit 1)
+    (in_bom yes) (on_board yes) (fields_autoplaced)
+    (property "Reference" "J7" (id 0) (at 224.7899 110.49 90)
       (effects (font (size 1.27 1.27)) (justify right))
     )
-    (property "Value" "Reserve_PinHeader" (id 1) (at 233.68 111.7599 90)
+    (property "Value" "Reserve_PinHeader" (id 1) (at 227.3299 110.49 90)
       (effects (font (size 1.27 1.27)) (justify right))
     )
-    (property "Footprint" "digikey-footprints:PinHeader_1x4_P2mm_Drill1mm" (id 2) (at 222.25 101.6 0)
-      (effects (font (size 1.524 1.524)) (justify left) hide)
-    )
-    (property "Datasheet" "" (id 3) (at 234.95 114.3 0)
+    (property "Footprint" "Connector_PinHeader_2.54mm:PinHeader_1x04_P2.54mm_Vertical" (id 2) (at 217.17 121.92 0)
+      (effects (font (size 1.524 1.524)) (justify left) hide)
+    )
+    (property "Datasheet" "" (id 3) (at 229.87 109.22 0)
       (effects (font (size 1.524 1.524)) hide)
     )
@@
     )
     (property "Value" "RotaryEncoder" (id 1) (at 138.43 102.87 0))
-    (property "Footprint" "" (id 2) (at 142.24 106.426 0)
+    (property "Footprint" "Rotary_Encoder:RotaryEncoder_Alps_EC11E-Switch_Vertical_H20mm" (id 2) (at 142.24 106.426 0)
       (effects (font (size 1.27 1.27)) hide)
     )
@@
     )
     (path "/c4ef8bf0-b9fa-40d3-ad8d-56b46e78b9a1"
-      (reference "J1") (unit 1) (value "Jack-DC") (footprint "")
+      (reference "J1") (unit 1) (value "Jack-DC") (footprint "Connector_BarrelJack:BarrelJack_Horizontal")
     )
     (path "/6e56f2a7-8754-4162-80c8-542615da19fa"
@@
     )
     (path "/d103ad51-1bb4-491e-8354-64c6e089e9f1"
-      (reference "J7") (unit 1) (value "Reserve_PinHeader") (footprint "digikey-footprints:PinHeader_1x4_P2mm_Drill1mm")
+      (reference "J7") (unit 1) (value "Reserve_PinHeader") (footprint "Connector_PinHeader_2.54mm:PinHeader_1x04_P2.54mm_Vertical")
     )
     (path "/02021ba7-4d1a-4846-a4b4-00321b415f7f"
@@
     )
     (path "/de986ad9-2077-4374-9035-245917b4b7a6"
-      (reference "SW1") (unit 1) (value "RotaryEncoder") (footprint "")
+      (reference "SW1") (unit 1) (value "RotaryEncoder") (footprint "Rotary_Encoder:RotaryEncoder_Alps_EC11E-Switch_Vertical_H20mm")
     )
     (path "/266f7da2-d095-4158-b55b-54efc0936b08"
-      (reference "SW2") (unit 1) (value "RotaryEncoder") (footprint "")
+      (reference "SW2") (unit 1) (value "RotaryEncoder") (footprint "Rotary_Encoder:RotaryEncoder_Alps_EC11E-Switch_Vertical_H20mm")
     )
     (path "/0aaa49ea-91cb-46ee-9047-c501634b853b"
-      (reference "SW3") (unit 1) (value "SW_DIP_x08") (footprint "")
+      (reference "SW3") (unit 1) (value "SW_DIP_x08") (footprint "Button_Switch_SMD:SW_DIP_SPSTx03_Slide_9.78x9.8mm_W8.61mm_P2.54mm")
     )
     (path "/b4b6c71b-c8e5-4172-96e6-29540545f271"
-      (reference "TP1") (unit 1) (value "TestPoint") (footprint "")
+      (reference "TP1") (unit 1) (value "TestPoint") (footprint "TestPoint:TestPoint_Pad_D2.0mm")
     )
     (path "/246ca8c3-d91c-4b19-a6a8-48a0cdc00a94"
-      (reference "TP2") (unit 1) (value "TestPoint") (footprint "")
+      (reference "TP2") (unit 1) (value "TestPoint") (footprint "TestPoint:TestPoint_Pad_D2.0mm")
     )
     (path "/0555d286-6d86-4552-94e8-d32676b671db"

Commit message: 5
Parts:
- C1: footprint (none) -> Capacitor_THT:CP_Radial_D5.0mm_P2.50mm
- C2, C3, C5: footprint (none) -> Capacitor_THT:C_Disc_D5.0mm_W2.5mm_P2.50mm
- C4, C6: footprint Capacitor_THT:C_Disc_D4.3mm_W1.9mm_P5.00mm -> Capacitor_THT:C_Disc_D3.8mm_W2.6mm_P2.50mm
- U1: footprint (none) -> Connector_PinHeader_2.54mm:PinHeader_1x04_P2.54mm_Vertical
- U2, U5: footprint (none) -> Motors:TB67S101ANG
- U3: footprint (none) -> Package_DIP:Tang_Nano_9K
- U4: footprint (none) -> LED_THT:OSL641501-ARA
Changed lines of the file:
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@@
       (effects (font (size 1.27 1.27)) (justify right top))
     )
-    (property "Footprint" "" (id 2) (at 44.1452 85.09 0)
+    (property "Footprint" "Capacitor_THT:C_Disc_D5.0mm_W2.5mm_P2.50mm" (id 2) (at 44.1452 85.09 0)
       (effects (font (size 1.27 1.27)) hide)
     )
@@
       (effects (font (size 1.27 1.27)) (justify left))
     )
-    (property "Footprint" "" (id 2) (at 66.04 22.86 0)
+    (property "Footprint" "Connector_PinHeader_2.54mm:PinHeader_1x04_P2.54mm_Vertical" (id 2) (at 66.04 22.86 0)
       (effects (font (size 1.27 1.27) italic) hide)
     )
@@
       (effects (font (size 1.27 1.27)) (justify right top))
     )
-    (property "Footprint" "" (id 2) (at 37.7952 55.88 0)
+    (property "Footprint" "Capacitor_THT:CP_Radial_D5.0mm_P2.50mm" (id 2) (at 37.7952 55.88 0)
       (effects (font (size 1.27 1.27)) hide)
     )
@@
     (property "Reference" "U2" (id 0) (at 77.47 53.34 0))
     (property "Value" "TB67S101ANG" (id 1) (at 77.47 55.88 0))
-    (property "Footprint" "" (id 2) (at 82.55 68.58 0)
+    (property "Footprint" "Motors:TB67S101ANG" (id 2) (at 82.55 68.58 0)
       (effects (font (size 1.524 1.524)) (justify left) hide)
     )
@@
     )
     (property "Value" "270p" (id 1) (at 62.23 91.4399 0))
-    (property "Footprint" "Capacitor_THT:C_Disc_D4.3mm_W1.9mm_P5.00mm" (id 2) (at 59.3852 93.98 0)
+    (property "Footprint" "Capacitor_THT:C_Disc_D3.8mm_W2.6mm_P2.50mm" (id 2) (at 59.3852 93.98 0)
       (effects (font (size 1.27 1.27)) hide)
     )
@@
     (property "Reference" "U4" (id 0) (at 236.22 101.6 0))
     (property "Value" "OSL641505-BB" (id 1) (at 236.22 99.06 0))
-    (property "Footprint" "" (id 2) (at 288.29 114.3 0)
+    (property "Footprint" "LED_THT:OSL641501-ARA" (id 2) (at 288.29 114.3 0)
       (effects (font (size 1.27 1.27)) hide)
     )
@@
       (effects (font (size 1.27 1.27)) (justify right top))
     )
-    (property "Footprint" "" (id 2) (at 44.1452 163.83 0)
+    (property "Footprint" "Capacitor_THT:C_Disc_D5.0mm_W2.5mm_P2.50mm" (id 2) (at 44.1452 163.83 0)
       (effects (font (size 1.27 1.27)) hide)
     )
@@
     (property "Reference" "U3" (id 0) (at 191.135 44.45 0))
     (property "Value" "TangNano9K" (id 1) (at 191.135 46.99 0))
-    (property "Footprint" "" (id 2) (at 222.25 45.72 0)
+    (property "Footprint" "Package_DIP:Tang_Nano_9K" (id 2) (at 222.25 45.72 0)
       (effects (font (size 1.27 1.27)) hide)
     )
@@
     (property "Reference" "U5" (id 0) (at 77.47 132.08 0))
     (property "Value" "TB67S101ANG" (id 1) (at 77.47 134.62 0))
-    (property "Footprint" "" (id 2) (at 82.55 147.32 0)
+    (property "Footprint" "Motors:TB67S101ANG" (id 2) (at 82.55 147.32 0)
       (effects (font (size 1.524 1.524)) (justify left) hide)
     )
@@
     )
     (property "Value" "270p" (id 1) (at 62.23 170.1799 0))
-    (property "Footprint" "Capacitor_THT:C_Disc_D4.3mm_W1.9mm_P5.00mm" (id 2) (at 59.3852 172.72 0)
+    (property "Footprint" "Capacitor_THT:C_Disc_D3.8mm_W2.6mm_P2.50mm" (id 2) (at 59.3852 172.72 0)
       (effects (font (size 1.27 1.27)) hide)
     )
@@
       (effects (font (size 1.27 1.27)) (justify right top))
     )
-    (property "Footprint" "" (id 2) (at 44.1452 55.88 0)
+    (property "Footprint" "Capacitor_THT:C_Disc_D5.0mm_W2.5mm_P2.50mm" (id 2) (at 44.1452 55.88 0)
       (effects (font (size 1.27 1.27)) hide)
     )
@@
     )
     (path "/1b203025-f9a0-4031-a2eb-97e7f134dcdb"
-      (reference "C1") (unit 1) (value "100μ") (footprint "")
+      (reference "C1") (unit 1) (value "100μ") (footprint "Capacitor_THT:CP_Radial_D5.0mm_P2.50mm")
     )
     (path "/f88607f0-b8ca-451c-9113-0f5bf3405953"
-      (reference "C2") (unit 1) (value "0.1μ") (footprint "")
+      (reference "C2") (unit 1) (value "0.1μ") (footprint "Capacitor_THT:C_Disc_D5.0mm_W2.5mm_P2.50mm")
     )
     (path "/03905288-6954-4141-9c45-1c11764a1ca3"
-      (reference "C3") (unit 1) (value "0.1μ") (footprint "")
+      (reference "C3") (unit 1) (value "0.1μ") (footprint "Capacitor_THT:C_Disc_D5.0mm_W2.5mm_P2.50mm")
     )
     (path "/3f9d012d-84b1-4698-b5f7-e431ed62cc93"
-      (reference "C4") (unit 1) (value "270p") (footprint "Capacitor_THT:C_Disc_D4.3mm_W1.9mm_P5.00mm")
+      (reference "C4") (unit 1) (value "270p") (footprint "Capacitor_THT:C_Disc_D3.8mm_W2.6mm_P2.50mm")
     )
     (path "/71d9e1f5-0827-4510-b811-be115d614ba5"
-      (reference "C5") (unit 1) (value "0.1μ") (footprint "")
+      (reference "C5") (unit 1) (value "0.1μ") (footprint "Capacitor_THT:C_Disc_D5.0mm_W2.5mm_P2.50mm")
     )
     (path "/ed01aafb-4cf2-4f1f-b1c7-63d4035ca6df"
-      (reference "C6") (unit 1) (value "270p") (footprint "Capacitor_THT:C_Disc_D4.3mm_W1.9mm_P5.00mm")
+      (reference "C6") (unit 1) (value "270p") (footprint "Capacitor_THT:C_Disc_D3.8mm_W2.6mm_P2.50mm")
     )
     (path "/c4ef8bf0-b9fa-40d3-ad8d-56b46e78b9a1"
@@
     )
     (path "/0555d286-6d86-4552-94e8-d32676b671db"
-      (reference "U1") (unit 1) (value "BP5293-5") (footprint "")
+      (reference "U1") (unit 1) (value "BP5293-5") (footprint "Connector_PinHeader_2.54mm:PinHeader_1x04_P2.54mm_Vertical")
     )
     (path "/3b4c24e8-0a83-40bc-8bf5-8923992c8f7f"
-      (reference "U2") (unit 1) (value "TB67S101ANG") (footprint "")
+      (reference "U2") (unit 1) (value "TB67S101ANG") (footprint "Motors:TB67S101ANG")
     )
     (path "/b07c7a86-f5e1-435b-90e8-dd8e473e3c0e"
-      (reference "U3") (unit 1) (value "TangNano9K") (footprint "")
+      (reference "U3") (unit 1) (value "TangNano9K") (footprint "Package_DIP:Tang_Nano_9K")
     )
     (path "/467c1fba-20c5-4c47-a5bb-8b74d3cc9c21"
-      (reference "U4") (unit 1) (value "OSL641505-BB") (footprint "")
+      (reference "U4") (unit 1) (value "OSL641505-BB") (footprint "LED_THT:OSL641501-ARA")
     )
     (path "/b5d87323-6270-4b62-ba18-02f5c393e6db"
-      (reference "U5") (unit 1) (value "TB67S101ANG") (footprint "")
-    )
-  )
+      (reference "U5") (unit 1) (value "TB67S101ANG") (footprint "Motors:TB67S101ANG")
+    )
+  )
