File: tangnano9k_motordriver.kicad_sch (KiCad schematic)
At the start: 30 parts, among them J1 Jack-DC, J2 Screw_Terminal_01x04, J3 Screw_Terminal_01x04, J4 Reserve, J5 Reserve, J6 Reserve, J7 Reserve_PinHeader, J8 Pmod, SW3 SW_DIP_x08, U1 BP5293-5, U2 TB67S101ANG, U3 TangNano9K, U4 OSL641505-BB, U5 TB67S101ANG

Commit message: 9
Parts:
- C1: footprint Capacitor_THT:CP_Radial_D5.0mm_P2.50mm -> Connector_PinHeader_2.54mm:PinHeader_1x05_P2.54mm_Vertical
- J7: footprint Connector_PinHeader_2.54mm:PinHeader_1x04_P2.54mm_Vertical -> Connector_PinHeader_2.54mm:PinHeader_1x05_P2.54mm_Vertical; symbol 455-1706-nd:455-1706-ND -> 455-2270-nd:455-2270-ND
Connections:
- net GND: now also J7.1
- net at U3.27 (PIN32_IOB15B_RGBINIT): now also J7.2; no longer J7.1
- net at U3.28 (PIN31_IOB15A_RGBINIT): now also J7.3; no longer J7.2
- net at U3.29 (PIN49_IOR24A_SPILCD_RS): now also J7.4; no longer J7.3
- net at U3.30 (PIN48_IOR24B_SPILCD_CS): now also J7.5; no longer J7.4
Changed lines of the file:
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@@
     (stroke (width 0) (type default) (color 0 0 0 0))
   )
-  (wire (pts (xy 218.44 119.38) (xy 218.44 128.27))
+  (wire (pts (xy 218.44 119.38) (xy 218.44 125.73))
     (stroke (width 0) (type default) (color 0 0 0 0))
   )
@@
     (stroke (width 0) (type default) (color 0 0 0 0))
   )
-  (wire (pts (xy 227.33 125.73) (xy 219.71 125.73))
+  (wire (pts (xy 227.33 123.19) (xy 219.71 123.19))
     (stroke (width 0) (type default) (color 0 0 0 0))
   )
@@
     (stroke (width 0) (type default) (color 0 0 0 0))
   )
+  (wire (pts (xy 224.79 128.27) (xy 227.33 128.27))
+    (stroke (width 0) (type default) (color 0 0 0 0))
+  )
   (wire (pts (xy 217.17 93.98) (xy 218.44 93.98))
     (stroke (width 0) (type default) (color 0 0 0 0))
@@
     (stroke (width 0) (type default) (color 0 0 0 0))
   )
-  (wire (pts (xy 220.98 114.3) (xy 220.98 123.19))
+  (wire (pts (xy 220.98 114.3) (xy 220.98 120.65))
     (stroke (width 0) (type default) (color 0 0 0 0))
   )
@@
     (stroke (width 0) (type default) (color 0 0 0 0))
   )
-  (wire (pts (xy 218.44 128.27) (xy 227.33 128.27))
+  (wire (pts (xy 218.44 125.73) (xy 227.33 125.73))
     (stroke (width 0) (type default) (color 0 0 0 0))
   )
@@
     (stroke (width 0) (type default) (color 0 0 0 0))
   )
-  (wire (pts (xy 219.71 125.73) (xy 219.71 116.84))
+  (wire (pts (xy 219.71 123.19) (xy 219.71 116.84))
     (stroke (width 0) (type default) (color 0 0 0 0))
   )
@@
     (stroke (width 0) (type default) (color 0 0 0 0))
   )
-  (wire (pts (xy 227.33 120.65) (xy 222.25 120.65))
+  (wire (pts (xy 227.33 118.11) (xy 222.25 118.11))
     (stroke (width 0) (type default) (color 0 0 0 0))
   )
@@
     (stroke (width 0) (type default) (color 0 0 0 0))
   )
-  (wire (pts (xy 222.25 120.65) (xy 222.25 111.76))
+  (wire (pts (xy 222.25 118.11) (xy 222.25 111.76))
     (stroke (width 0) (type default) (color 0 0 0 0))
   )
@@
     (stroke (width 0) (type default) (color 0 0 0 0))
   )
-  (wire (pts (xy 220.98 123.19) (xy 227.33 123.19))
+  (wire (pts (xy 220.98 120.65) (xy 227.33 120.65))
     (stroke (width 0) (type default) (color 0 0 0 0))
   )
@@
       (effects (font (size 1.27 1.27)) (justify right top))
     )
-    (property "Footprint" "Capacitor_THT:CP_Radial_D5.0mm_P2.50mm" (id 2) (at 37.7952 55.88 0)
+    (property "Footprint" "Connector_PinHeader_2.54mm:PinHeader_1x05_P2.54mm_Vertical" (id 2) (at 37.7952 55.88 0)
       (effects (font (size 1.27 1.27)) hide)
     )
@@
     (pin "1")
     (pin "2")
+  )
+  (symbol (lib_id "power:GND") (at 224.79 128.27 0) (unit 1)
+    (in_bom yes) (on_board yes) (fields_autoplaced)
+    (property "Reference" "#PWR0111" (id 0) (at 224.79 134.62 0)
+      (effects (font (size 1.27 1.27)) hide)
+    )
+    (property "Value" "GND" (id 1) (at 224.79 133.35 0))
+    (property "Footprint" "" (id 2) (at 224.79 128.27 0)
+      (effects (font (size 1.27 1.27)) hide)
+    )
+    (property "Datasheet" "" (id 3) (at 224.79 128.27 0)
+      (effects (font (size 1.27 1.27)) hide)
+    )
+    (pin "1")
   )
   (symbol (lib_id "power:GND") (at 148.59 130.81 0) (unit 1)
@@
     (pin "4")
   )
-  (symbol (lib_name "455-1706-ND_1") (lib_id "455-1706-nd:455-1706-ND") (at 229.87 128.27 90) (unit 1)
+  (symbol (lib_id "455-2270-nd:455-2270-ND") (at 229.87 128.27 90) (unit 1)
     (in_bom yes) (on_board yes)
     (property "Reference" "J7" (id 0) (at 228.6 130.81 90)
@@
       (effects (font (size 1.27 1.27)) (justify right))
     )
-    (property "Footprint" "Connector_PinHeader_2.54mm:PinHeader_1x04_P2.54mm_Vertical" (id 2) (at 217.17 135.89 0)
-      (effects (font (size 1.524 1.524)) (justify left) hide)
-    )
-    (property "Datasheet" "" (id 3) (at 229.87 123.19 0)
+    (property "Footprint" "Connector_PinHeader_2.54mm:PinHeader_1x05_P2.54mm_Vertical" (id 2) (at 222.25 115.57 0)
+      (effects (font (size 1.524 1.524)) (justify left) hide)
+    )
+    (property "Datasheet" "" (id 3) (at 234.95 128.27 0)
       (effects (font (size 1.524 1.524)) hide)
     )
@@
     (pin "3")
     (pin "4")
+    (pin "5")
   )
   (symbol (lib_id "Device:RotaryEncoder_Switch") (at 138.43 124.46 0) (mirror y) (unit 1)
@@
       (reference "#PWR0110") (unit 1) (value "+3.3V") (footprint "")
     )
+    (path "/5cf04c0c-ddd6-454b-b71a-cf4b34a29abb"
+      (reference "#PWR0111") (unit 1) (value "GND") (footprint "")
+    )
     (path "/1b203025-f9a0-4031-a2eb-97e7f134dcdb"
-      (reference "C1") (unit 1) (value "100μ") (footprint "Capacitor_THT:CP_Radial_D5.0mm_P2.50mm")
+      (reference "C1") (unit 1) (value "100μ") (footprint "Connector_PinHeader_2.54mm:PinHeader_1x05_P2.54mm_Vertical")
     )
     (path "/f88607f0-b8ca-451c-9113-0f5bf3405953"
@@
     )
     (path "/d103ad51-1bb4-491e-8354-64c6e089e9f1"
-      (reference "J7") (unit 1) (value "Reserve_PinHeader") (footprint "Connector_PinHeader_2.54mm:PinHeader_1x04_P2.54mm_Vertical")
+      (reference "J7") (unit 1) (value "Reserve_PinHeader") (footprint "Connector_PinHeader_2.54mm:PinHeader_1x05_P2.54mm_Vertical")
     )
     (path "/1a2a9b14-1d5a-4abc-b1b0-6f3bbdb6e73e"

Commit message: ver02
Parts:
- removed J7: Reserve_PinHeader, Connector_PinHeader_2.54mm:PinHeader_1x05_P2.54mm_Vertical, symbol 455-2270-nd:455-2270-ND
- removed TP1, TP2: TestPoint, TestPoint:TestPoint_Pad_D2.0mm, symbol Connector:TestPoint
- added C7: 0.1μ, Capacitor_THT:C_Disc_D5.0mm_W2.5mm_P2.50mm, symbol Device:C
- added C8, C9: 1μ, Capacitor_THT:C_Disc_D5.0mm_W2.5mm_P2.50mm, symbol Device:C
- added DS1: A-551SRD-AG_W, samactech:DIPS1524W51P254L1270H825Q10N, symbol samacsys:A-551SRD-AG_W
- added F1: Polyfuse, Fuse:Fuse_Bourns_MF-RHT300, symbol Device:Polyfuse
- added JP1, JP2, JP3, JP4, JP5, JP6, JP7, JP8, JP9: SolderJumper_2_Open, Jumper:SolderJumper-2_P1.3mm_Open_TrianglePad1.0x1.5mm, symbol Jumper:SolderJumper_2_Open
- added R7, R8: 100k, Resistor_THT:R_Axial_DIN0207_L6.3mm_D2.5mm_P7.62mm_Horizontal, symbol Device:R
- C1: footprint Connector_PinHeader_2.54mm:PinHeader_1x05_P2.54mm_Vertical -> Capacitor_THT:CP_Radial_D8.0mm_P2.50mm
- renumbered J8 to J4, J4 to Pin1, J5 to Pin2, J6 to Pin3, Rotary_SW2 to Rotary_SW1, Rotary_SW1 to Rotary_SW2
Connections:
- net A_1: now also U3.23 (HDMI_CK_N), JP7.1 (A); no longer U3.22 (PIN57_IOR13A_RGB_G5)
- net A_2: no longer Rotary_SW1.A, U3.18 (PIN53_IOR15B_RGB_B4)
- net B_1: now also U3.19 (PIN54_IOR15A_RGB_B3), JP6.1 (A); no longer U3.24 (HDMI_CK_P)
- net B_2: no longer Rotary_SW1.B, U3.20 (PIN55_IOR14B_RGB_G7)
- net GND: now also C7.2, C8.2, C9.2
- net PHASEA_1: now also Pin2.4, U3.5 (PIN25_IOB8A); no longer Pin1.4, U3.1 (PIN38_IOB31B_TF_CS)
- net PHASEA_2: now also U3.21 (PIN56_IOR14A_RGB_G6); no longer Pin2.4, U3.5 (PIN25_IOB8A)
- net PHASEB_1: now also Pin1.1, U3.4 (PIN39_IOB33A_TF_MISO); no longer Pin1.3, U3.2 (PIN37_IOB31A_TF_MOSI)
- net PHASEB_2: now also U3.20 (PIN55_IOR14B_RGB_G7); no longer Pin2.3, U3.6 (PIN26_IOB8B)
- net STANBY_1: now also Pin1.4, U3.1 (PIN38_IOB31B_TF_CS); no longer Pin1.1, U3.4 (PIN39_IOB33A_TF_MISO)
- net STANBY_2: now also U3.17 (PIN51_IOR17B_RGB_B5); no longer Pin2.1, U3.8 (PIN28_IOB11B)
- net VREF_1: now also C8.1, R7.1; no longer Pin1.2, U3.3 (PIN36_IOB29B_TF_SCLK)
- net VREF_2: now also C9.1, R8.1; no longer Pin2.2, U3.7 (PIN27_IOB11A)
- net VM: now reaches C1.1, C2.1, R2.1, R3.2, R5.1, R6.2, U2.7 (VM), U5.7 (VM)
- net VM: now also C7.1, F1.2; no longer J1.1, U1.1 (VIN)
- net Reserve_b: now reaches Pin3.1
- net Reserve_b: now also U3.9 (PIN29_IOB13A); no longer U3.21 (PIN56_IOR14A_RGB_G6)
- net INA1: now reaches Pin3.2
- net INA1: now also U2.12 (INA1), U3.10 (PIN30_IOB13B); no longer U3.9 (PIN29_IOB13A)
- net at Rotary_SW1.S1: now also U3.48 (PIN63_IOR5A_RGBINIT); no longer U3.19 (PIN54_IOR15A_RGB_B3)
- net R5: now reaches U3.32 (HDMI_D0_N), U4.1 (R5)
- net C1: now reaches U3.11 (PIN33_IOB23A_RGB_DE)
- net C1: now also U4.13 (C1), DS1.4 (C_C); no longer U4.10 (C4)
- net C6: now reaches U4.11 (C6)
- net C6: now also U3.28 (PIN31_IOB15A_RGBINIT), DS1.2 (C_D); no longer U3.12 (PIN34_IOB23B_RGB_VS)
- net C7: now reaches U3.13 (PIN40_IOB33B_RGB_HS)
- net C7: now also U4.15 (C7), DS1.5 (C_DP); no longer U4.12 (R4)
- net C8: now reaches U3.14 (PIN35_IOB29A_RGB_CK)
- net C8: now also U4.16 (C8), DS1.6 (C_B); no longer U4.13 (C1)
- net at U3.15 (PIN41_IOB41A_RGB_B7): now also Rotary_SW1.A; no longer U4.14 (R2)
- net at U3.16 (PIN42_IOB41B_RGB_B6): now also Rotary_SW1.B; no longer U4.15 (C7)
- net R7: now reaches U3.33 (HDMI_D0_P), U4.2 (R7)
- net C2: now reaches U3.34 (HDMI_D1_N), U4.3 (C2)
- net C2: now also DS1.9 (C_F)
- net C3: now reaches U3.35 (HDMI_D1_P), U4.4 (C3)
- net C3: now also DS1.10 (C_G)
- net R8: now reaches U3.36 (HDMI_D2_N), U4.5 (R8)
- net C5: now reaches U3.37 (HDMI_D2_P), U4.6 (C5)
- net C5: now also DS1.7 (C_A)
- net R6: now reaches U3.38 (PIN76_IOT37B_SPILCD_MCLK), U4.7 (R6)
- net R3: now reaches U3.39 (PIN77_IOT37A_SPILCD_MO), U4.8 (R3)
- net R1: now reaches U4.9 (R1)
- net R1: now also U3.30 (PIN48_IOR24B_SPILCD_CS); no longer U3.10 (PIN30_IOB13B)
- net at Rotary_SW2.S1: now also U3.22 (PIN57_IOR13A_RGB_G5), JP8.1 (A); no longer U3.23 (HDMI_CK_N)
- net R4: now reaches U3.27 (PIN32_IOB15B_RGBINIT)
- net R4: now also U4.12 (R4)
- net C4: now reaches U3.29 (PIN49_IOR24A_SPILCD_RS)
- net C4: now also U4.10 (C4), DS1.1 (C_E)
- new net: F1.1, J1.1, U1.1 (VIN)
- new net: J4.8 (10), SW3.1, U3.40 (PIN79_IOT12B_1V8)
- new net: J4.6 (9), SW3.2, U3.41 (PIN80_IOT12A_1V8)
- new net: J4.5 (3), SW3.3, U3.42 (PIN81_IOT11B_1V8)
- new net: J4.7 (4), SW3.4, U3.43 (PIN82_IOT11A_1V8)
- new net: J4.9 (5), SW3.5, U3.44 (PIN83_IOT10B_1V8)
- new net: J4.11 (6), SW3.6, U3.45 (PIN84_IOT10A_1V8)
- new net: J4.12, SW3.7, U3.46 (PIN85_IOT8B_1V8)
- new net: J4.10 (11), SW3.8, U3.47 (PIN86_IOT8A_BL_PWM_1V8)
- new net: JP5.1 (A), JP9.1 (A), U3.18 (PIN53_IOR15B_RGB_B4)
- new net: R8.2, U3.24 (HDMI_CK_P)
- new net: DS1.3 (COMMON_ANODE_1), DS1.8 (COMMON_ANODE_2), JP9.2 (B)
- new net INA1_2: JP1.2 (B), JP8.2 (B), U5.12 (INA1)
- new net INA2: Pin2.3, U2.13 (INA2), U3.6 (PIN26_IOB8B)
- new net INA2_2: JP2.2 (B), JP7.2 (B), U5.13 (INA2)
- new net INB1: Pin1.2, U2.16 (INB1), U3.3 (PIN36_IOB29B_TF_SCLK)
- new net INB1_2: JP3.2 (B), JP6.2 (B), U5.16 (INB1)
- new net INB2: Pin1.3, U2.17 (INB2), U3.2 (PIN37_IOB31A_TF_MOSI)
- new net INB2_2: JP4.2 (B), JP5.2 (B), U5.17 (INB2)
- new net R2: U3.12 (PIN34_IOB23B_RGB_VS), U4.14 (R2)
- new net Reserve_a: Pin2.1, U3.8 (PIN28_IOB11B)
- new net VCC_1: C3.1, R1.1, U2.8 (VCC)
- new net VCC_2: C5.1, JP1.1 (A), JP2.1 (A), JP3.1 (A), JP4.1 (A), R4.1, U5.8 (VCC)
- new net VREF_PWM_1: Pin2.2, R7.2, U3.7 (PIN27_IOB11A)
Other:
- moved on the sheet: J4, Pin1, Pin2, Pin3, R6, Rotary_SW1, Rotary_SW2, SW3, U4

Commit message: 17
Connections:
- net C1: no longer DS1.4 (C_C), U3.11 (PIN33_IOB23A_RGB_DE), U4.13 (C1)
- net C2: no longer DS1.9 (C_F), U3.34 (HDMI_D1_N), U4.3 (C2)
- net C3: no longer DS1.10 (C_G), U3.35 (HDMI_D1_P), U4.4 (C3)
- net C4: no longer DS1.1 (C_E), U3.29 (PIN49_IOR24A_SPILCD_RS), U4.10 (C4)
- net C5: no longer DS1.7 (C_A), U3.37 (HDMI_D2_P), U4.6 (C5)
- net C6: no longer DS1.2 (C_D), U3.28 (PIN31_IOB15A_RGBINIT), U4.11 (C6)
- net C7: no longer DS1.5 (C_DP), U3.13 (PIN40_IOB33B_RGB_HS), U4.15 (C7)
- net C8: no longer DS1.6 (C_B), U3.14 (PIN35_IOB29A_RGB_CK), U4.16 (C8)
- net R2: no longer U3.12 (PIN34_IOB23B_RGB_VS), U4.14 (R2)
- net R3: no longer U3.39 (PIN77_IOT37A_SPILCD_MO), U4.8 (R3)
- net R4: no longer U3.27 (PIN32_IOB15B_RGBINIT), U4.12 (R4)
- net R5: no longer U3.32 (HDMI_D0_N), U4.1 (R5)
- net R6: no longer U3.38 (PIN76_IOT37B_SPILCD_MCLK), U4.7 (R6)
- net R7: no longer U3.33 (HDMI_D0_P), U4.2 (R7)
- net R8: no longer U3.36 (HDMI_D2_N), U4.5 (R8)
- net R9: now reaches DS1.3 (C_ANODE_1), DS1.8 (C_ANODE_2), JP9.2 (B)
- new net: U3.32 (HDMI_D0_N), U4.1 (R5)
- new net: DS1.1 (C_E), U3.29 (PIN49_IOR24A_SPILCD_RS), U4.10 (C4)
- new net: DS1.2 (C_D), U3.28 (PIN31_IOB15A_RGBINIT), U4.11 (C6)
- new net: U3.27 (PIN32_IOB15B_RGBINIT), U4.12 (R4)
- new net: DS1.4 (C_C), U3.11 (PIN33_IOB23A_RGB_DE), U4.13 (C1)
- new net: U3.12 (PIN34_IOB23B_RGB_VS), U4.14 (R2)
- new net: DS1.5 (C_DP), U3.13 (PIN40_IOB33B_RGB_HS), U4.15 (C7)
- new net: DS1.6 (C_B), U3.14 (PIN35_IOB29A_RGB_CK), U4.16 (C8)
- new net: U3.33 (HDMI_D0_P), U4.2 (R7)
- new net: DS1.9 (C_F), U3.34 (HDMI_D1_N), U4.3 (C2)
- new net: DS1.10 (C_G), U3.35 (HDMI_D1_P), U4.4 (C3)
- new net: U3.36 (HDMI_D2_N), U4.5 (R8)
- new net: DS1.7 (C_A), U3.37 (HDMI_D2_P), U4.6 (C5)
- new net: U3.38 (PIN76_IOT37B_SPILCD_MCLK), U4.7 (R6)
- new net: U3.39 (PIN77_IOT37A_SPILCD_MO), U4.8 (R3)
Other:
- moved on the sheet: DS1, J4, JP9, SW3, U3, U4

Commit message: 6
Parts:
- added JP10, JP11, JP12, JP13, JP14: SolderJumper_2_Open, Library:SolderJumper_Register_Horizontal, symbol Jumper:SolderJumper_2_Open
- added JP15, JP16, JP17: SolderJumper_2_Open, Library:SolderJumper_Register, symbol Jumper:SolderJumper_2_Open
- added TP1: TestPoint, TestPoint:TestPoint_THTPad_1.5x1.5mm_Drill0.7mm, symbol Connector:TestPoint
- added TP2: TestPoint, TestPoint:TestPoint_Pad_1.5x1.5mm, symbol Connector:TestPoint
- renumbered C7 to C1, C1 to C2, C2 to C3, C3 to C4, C4 to C6, C6 to C7, R4 to R2, R2 to R3, R5 to R4, R7 to R5, R8 to R6, R6 to R7, R3 to R8, Rotary_SW2 to Rotary_SW1, Rotary_SW1 to Rotary_SW2, SW3 to SW1, U5 to U3, U3 to U4, U4 to U5
Connections:
- net R1: now also JP15.2 (B); no longer U4.30 (PIN48_IOR24B_SPILCD_CS)
- net VREF_1: now also TP1.1
- net VREF_2: now also TP2.1
- net at U5.1 (R5): now also JP10.2 (B); no longer U4.32 (HDMI_D0_N)
- net at U4.27 (PIN32_IOB15B_RGBINIT): now also JP16.1 (A); no longer U5.12 (R4)
- net at U4.12 (PIN34_IOB23B_RGB_VS): now also JP17.1 (A); no longer U5.14 (R2)
- net at U5.2 (R7): now also JP11.2 (B); no longer U4.33 (HDMI_D0_P)
- net at DS1.10 (C_G), U4.35 (HDMI_D1_P): now also JP12.1 (A); no longer U5.4 (C3)
- net at U5.7 (R6): now also JP13.2 (B); no longer U4.38 (PIN76_IOT37B_SPILCD_MCLK)
- net at U5.8 (R3): now also JP14.2 (B); no longer U4.39 (PIN77_IOT37A_SPILCD_MO)
- new net: JP16.2 (B), U5.12 (R4)
- new net: JP17.2 (B), U5.14 (R2)
- new net: JP12.2 (B), U5.4 (C3)
- new net: JP11.1 (A), U4.33 (HDMI_D0_P)
- new net: JP15.1 (A), U4.30 (PIN48_IOR24B_SPILCD_CS)
- new net: JP14.1 (A), U4.39 (PIN77_IOT37A_SPILCD_MO)
- new net: JP13.1 (A), U4.38 (PIN76_IOT37B_SPILCD_MCLK)
- new net: JP10.1 (A), U4.32 (HDMI_D0_N)
- no-connect marks 2 -> 4
Other:
- moved on the sheet: Pin1, Pin2, Pin3, U4

Commit message: 1
Connections:
- net +3.3V: now also J4.11 (6), J4.12; no longer J4.1
- net GND: now also J4.9 (5); no longer J4.3 (2)
- net at SW1.1, U4.40 (PIN79_IOT12B_1V8): now also J4.4 (8); no longer J4.8 (10)
- net at SW1.2, U4.41 (PIN80_IOT12A_1V8): now also J4.2 (7); no longer J4.6 (9)
- net at SW1.3, U4.42 (PIN81_IOT11B_1V8): now also J4.1; no longer J4.5 (3)
- net at SW1.4, U4.43 (PIN82_IOT11A_1V8): now also J4.3 (2); no longer J4.7 (4)
- net at SW1.5, U4.44 (PIN83_IOT10B_1V8): now also J4.5 (3); no longer J4.9 (5)
- net at SW1.6, U4.45 (PIN84_IOT10A_1V8): now also J4.7 (4); no longer J4.11 (6)
- net at SW1.7, U4.46 (PIN85_IOT8B_1V8): now also J4.8 (10); no longer J4.12
- net at SW1.8, U4.47 (PIN86_IOT8A_BL_PWM_1V8): now also J4.6 (9); no longer J4.10 (11)
- no-connect marks 4 -> 2
