File: tangnano9k_motordriver.kicad_pcb (KiCad board)
At the start: 2 copper layers, 115.6 x 92.7 mm, 30 parts, among them J1 Jack-DC, J2 Screw_Terminal_01x04, J3 Screw_Terminal_01x04, J4 Reserve, J5 Reserve, J6 Reserve, J7 Reserve_PinHeader, J8 Pmod, SW3 SW_DIP_x08, U1 BP5293-5, U2 TB67S101ANG, U3 TangNano9K, U4 OSL641505-BB, U5 TB67S101ANG

Commit message: 7
Parts:
- moved R4 26.4 mm to (86.4, 132.1), turned to -90 degrees
- moved R1 25.7 mm to (86.4, 94.0), turned to -90 degrees
- moved C2 24.1 mm to (86.4, 66.0), turned to -90 degrees
- moved U1 15.3 mm to (91.4, 66.0)
- moved C3 14.8 mm to (86.4, 90.2), turned to 90 degrees
- moved C4 13.7 mm to (86.4, 83.8)
- moved C5 11.7 mm to (86.4, 124.5)
- moved U5 10.8 mm to (72.4, 114.3)
- moved Rotary_SW1 10.2 mm to (94.3, 134.7)
- moved C6 9.18 mm to (86.4, 119.3)
- moved J2 8.07 mm to (64.8, 83.8)
- moved Rotary_SW2 7.99 mm to (116.3, 134.7)
- moved U2 7.66 mm to (72.4, 82.5)
- moved J3 7.62 mm to (64.8, 118.1)
- moved C1 6.48 mm to (81.3, 66.1)
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Other:
- board size 115.6 x 92.7 mm -> 107.9 x 86.4 mm

Commit message: 8
Parts:
- moved R5 31.9 mm to (86.4, 141.0)
- moved R3 28.0 mm to (71.1, 80.0), turned to 0 degrees
- moved R2 27.7 mm to (91.4, 102.9)
- moved U5 22.3 mm to (66.7, 135.9), turned to 90 degrees
- moved R6 22.2 mm to (71.1, 118.1), turned to 0 degrees
- moved J4 18.2 mm to (90.2, 58.4)
- moved J5 18.2 mm to (90.2, 68.6)
- moved J6 18.2 mm to (90.2, 73.7)
- moved U3 17.7 mm to (95.2, 50.8)
- moved J2 16.5 mm to (64.8, 67.3)
- moved U2 16.3 mm to (66.6, 97.8), turned to 90 degrees
- moved J8 15.6 mm to (148.0, 62.2)
- moved C1 14.0 mm to (80.0, 52.1)
- moved J1 14.0 mm to (73.7, 52.1)
- moved J3 12.7 mm to (64.8, 105.4)
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Routing:
- net GND: track 0.00 -> 152.5 mm, vias 0 -> 3
- net /VREF_2: track 0.00 -> 91.0 mm, vias 0 -> 1
- net /PHASEA_2: track 0.00 -> 90.1 mm, vias 0 -> 1
- net /STANBY_2: track 0.00 -> 87.7 mm, vias 0 -> 3
- net /PHASEB_2: track 0.00 -> 87.4 mm, vias 0 -> 1
- net Net-(C1-Pad1): track 0.00 -> 86.8 mm
- net Net-(C5-Pad1): track 0.00 -> 36.7 mm
- net /B_1: track 0.00 -> 33.6 mm
- net Net-(J6-Pad1): track 0.00 -> 33.0 mm
- net Net-(J3-Pad3): track 0.00 -> 28.3 mm, vias 0 -> 1
- net Net-(C6-Pad1): track 0.00 -> 27.5 mm
- net Net-(J2-Pad3): track 0.00 -> 27.2 mm, vias 0 -> 1
- net Net-(J3-Pad4): track 0.00 -> 26.2 mm
- net Net-(J2-Pad4): track 0.00 -> 26.1 mm
- net Net-(J2-Pad1): track 0.00 -> 24.3 mm
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Other:
- board size 107.9 x 86.4 mm -> 99.8 x 99.8 mm

Commit message: 9
Parts:
- C1: footprint Capacitor_THT:CP_Radial_D5.0mm_P2.50mm -> Connector_PinHeader_2.54mm:PinHeader_1x05_P2.54mm_Vertical
- J7: footprint Connector_PinHeader_2.54mm:PinHeader_1x04_P2.54mm_Vertical -> Connector_PinHeader_2.54mm:PinHeader_1x05_P2.54mm_Vertical
Connections:
- J7 pad 1: Net-(J7-Pad1) -> GND
- U3 pad 27: Net-(J7-Pad1) -> Net-(J7-Pad2)
- U3 pad 28: Net-(J7-Pad2) -> Net-(J7-Pad3)
- U3 pad 29: Net-(J7-Pad3) -> Net-(J7-Pad4)
- U3 pad 30: Net-(J7-Pad4) -> Net-(J7-Pad5)
Routing:
- net GND: track 152.5 -> 232.3 mm
- net Net-(Rotary_SW2-PadS1): track 0.00 -> 79.1 mm, vias 0 -> 2
- net /B_2: track 0.00 -> 59.7 mm, vias 0 -> 3
- net /A_2: track 0.00 -> 58.6 mm, vias 0 -> 3
- net Net-(Rotary_SW1-PadS1): track 0.00 -> 49.9 mm, vias 0 -> 2
- net /A_1: track 0.00 -> 32.6 mm
- net Net-(C1-Pad1): track 86.8 -> 102.1 mm

Commit message: 10
Parts:
- added ?: , , F.Cu at (131.4, 50.8)
- C1: footprint Connector_PinHeader_2.54mm:PinHeader_1x05_P2.54mm_Vertical -> Capacitor_THT:CP_Radial_D6.3mm_P2.50mm
- moved C2 2.54 mm to (73.7, 61.6), turned to 180 degrees
- moved TP2 2.54 mm to (118.1, 124.5)
- moved U1 2.54 mm to (80.0, 61.6)
Routing:
- net GND: track 232.3 -> 437.3 mm, vias 3 -> 4
- net +3.3V: track 0.00 -> 135.9 mm, vias 0 -> 2
- net Net-(J8-Pad12): track 0.00 -> 133.5 mm, vias 0 -> 3
- net Net-(J8-Pad11): track 0.00 -> 130.5 mm
- net Net-(J8-Pad10): track 0.00 -> 126.8 mm, vias 0 -> 3
- net Net-(J8-Pad8): track 0.00 -> 120.1 mm, vias 0 -> 3
- net Net-(J8-Pad9): track 0.00 -> 115.9 mm
- net Net-(J8-Pad6): track 0.00 -> 114.0 mm, vias 0 -> 1
- net Net-(J8-Pad7): track 0.00 -> 113.6 mm, vias 0 -> 2
- net Net-(J8-Pad5): track 0.00 -> 110.0 mm, vias 0 -> 2
- net +5V: track 0.00 -> 90.6 mm, vias 0 -> 1
- net Net-(J7-Pad2): track 0.00 -> 80.6 mm, vias 0 -> 2
- net Net-(J7-Pad3): track 0.00 -> 77.2 mm, vias 0 -> 2
- net Net-(U3-Pad10): track 0.00 -> 76.1 mm
- net Net-(U3-Pad11): track 0.00 -> 74.0 mm
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Other:
- board text added: "3V3"
- board text added: "5V"
- board text added: "A"
- board text added: "B"
- board text added: "GND"
- board text added: "STB"

Commit message: 11
Routing:
- net GND: track 437.3 -> 443.0 mm, vias 4 -> 2
- net Net-(C1-Pad1): track 152.7 -> 149.7 mm
- added copper zone on B.Cu, net GND
- added copper zone on F.Cu, net GND
Other:
- board text added: "(25)"
- board text added: "(26)"
- board text added: "(27)"
- board text added: "(28)"
- board text added: "(29)"
- board text added: "(30)"
- board text added: "(31)"
- board text added: "(32)"
- board text added: "(33)"
- board text added: "(34)"
- board text added: "(35)"
- board text added: "(36)"
- board text added: "(37)"
- board text added: "(38)"
- board text added: "(39)"
- board text added: "(40)"
- board text added: "(41)"
- board text added: "(42)"
- board text added: "(48)"
- board text added: "(49)"
- board text added: "(51)"
- board text added: "(53)"
- board text added: "(54)"
- board text added: "(55)"
- board text added: "(56)"
- board text added: "(57)"
- board text added: "(63)"
- board text added: "(68)"
- board text added: "(69)"
- board text added: "(70)"
- board text added: "(71)"
- board text added: "(72)"
- board text added: "(73)"
- board text added: "(74)"
- board text added: "(75)"
- board text added: "(76)"
- board text added: "(77)"
- board text added: "(79)"
- board text added: "(80)"
- board text added: "(81)"
- board text added: "(82)"
- board text added: "(83)"
- board text added: "(84)"
- board text added: "(85)"
- board text added: "(86)"
- board text added: "< ↑HDMI >"
- board text added: "< ↑USB >"
- board text added: "A+"
- board text added: "A-"
- board text added: "B+"
- board text added: "B-"
- board text added: "DC IN"
- board text added: "IN 7～26V"
- board text added: "INA1"
- board text added: "INA2"
- board text added: "INB1"
- board text added: "INB2"
- board text added: "OSCM"
- board text added: "OUTA+"
- board text added: "OUTA-"
- board text added: "OUTB+"
- board text added: "OUTB-"
- board text added: "RSA"
- board text added: "RSB"
- board text added: "SW"
- board text added: "Tang Nano 9K"
- board text added: "VCC"
- board text added: "VM"
- board text added: "VREFA"
- board text added: "VREFB"
- board text added: "[ OSL641501 -ARA ]"
- board text added: "[ TB67S101ANG ]"

Commit message: 12
Routing:
- net GND: track 443.0 -> 411.1 mm, vias 2 -> 10
- net Net-(C1-Pad1): track 149.7 -> 157.7 mm, vias 1 -> 13
- net Net-(TP1-Pad1): track 8.95 -> 13.4 mm
- net /PHASEA_1: track 52.9 -> 52.4 mm, vias 3 -> 2
- added copper zone on B.Cu, net Net-(C1-Pad1)
- added copper zone on F.Cu, net Net-(C1-Pad1)

Commit message: 13
Parts:
- added G***: LOGO, Library:logo_kamo, F.Cu at (151.1, 79.4)
- added REF**: MountingHole_2.7mm_M2.5, MountingHole:MountingHole_2.7mm_M2.5, F.Cu at (156.8, 70.5)
- added REF**: MountingHole_2.7mm_M2.5, MountingHole:MountingHole_2.7mm_M2.5, F.Cu at (63.8, 144.0)
- added REF**: MountingHole_2.7mm_M2.5, MountingHole:MountingHole_2.7mm_M2.5, F.Cu at (158.0, 144.1)
- added REF**: MountingHole_2.7mm_M2.5, MountingHole:MountingHole_2.7mm_M2.5, F.Cu at (64.4, 60.9)
Other:
- board text added: "Motor Driver Board for Tang Nano 9K Ver 0.1"
- board text added: "Sugamo"

Commit message: 14
Routing:
- net GND: vias 10 -> 35
Other:
- board text added: "[ OSL641501-ARA ]"
- board text removed: "[ OSL641501 -ARA ]"
