File: tangnano9k_motordriver.kicad_pcb (KiCad board)
At the start: 2 copper layers, 99.8 x 99.8 mm, 58 parts, among them J1 Jack-DC, J2 Screw_Terminal_01x04, J3 Screw_Terminal_01x04, J4 Pmod, SW1 SW_DIP_x08, U1 BP5293-5, U2 TB67S101ANG, U3 TB67S101ANG, U4 TangNano9K, U5 OSL641505-BB

Commit message: 6
Other:
- board text added: "Motor Driver Board for Tang Nano 9K Ver 0.3"
- board text removed: "Motor Driver Board for Tang Nano 9K Ver 0.2"
Changed lines of the file:
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@@
     (effects (font (size 1 1) (thickness 0.15)))
   )
-  (gr_text "Motor Driver Board for Tang Nano 9K Ver 0.2" (at 136.525 145.415) (layer "F.SilkS")
+  (gr_text "Motor Driver Board for Tang Nano 9K Ver 0.3" (at 136.525 145.415) (layer "F.SilkS")
     (effects (font (size 1 1) (thickness 0.15)))
   )
