File: tangnano9k_motordriver.kicad_pcb (KiCad board)
At the start: 2 copper layers, 99.8 x 99.8 mm, 58 parts, among them J1 Jack-DC, J2 Screw_Terminal_01x04, J3 Screw_Terminal_01x04, J4 Pmod, SW1 SW_DIP_x08, U1 BP5293-5, U2 TB67S101ANG, U3 TB67S101ANG, U4 TangNano9K, U5 OSL641505-BB

Commit message: 1
Parts:
- moved REF** 0.51 mm to (157.2, 49.8)
Connections:
- J4 pad 1: +3.3V -> Net-(SW1-Pad3)
- J4 pad 10: Net-(J4-Pad10) -> unconnected-(J4-Pad10)
- J4 pad 11: Net-(J4-Pad11) -> +3.3V
- J4 pad 12: Net-(J4-Pad12) -> +3.3V
- J4 pad 2: unconnected-(J4-Pad2) -> Net-(SW1-Pad2)
- J4 pad 3: GND -> Net-(SW1-Pad4)
- J4 pad 4: unconnected-(J4-Pad4) -> Net-(SW1-Pad1)
- J4 pad 5: Net-(J4-Pad5) -> Net-(SW1-Pad5)
- J4 pad 6: Net-(J4-Pad6) -> Net-(SW1-Pad8)
- J4 pad 7: Net-(J4-Pad7) -> Net-(SW1-Pad6)
- J4 pad 8: Net-(J4-Pad8) -> Net-(SW1-Pad7)
- J4 pad 9: Net-(J4-Pad9) -> GND
- SW1 pad 1: Net-(J4-Pad8) -> Net-(SW1-Pad1)
- SW1 pad 2: Net-(J4-Pad6) -> Net-(SW1-Pad2)
- SW1 pad 3: Net-(J4-Pad5) -> Net-(SW1-Pad3)
- SW1 pad 4: Net-(J4-Pad7) -> Net-(SW1-Pad4)
- SW1 pad 5: Net-(J4-Pad9) -> Net-(SW1-Pad5)
- SW1 pad 6: Net-(J4-Pad11) -> Net-(SW1-Pad6)
- SW1 pad 7: Net-(J4-Pad12) -> Net-(SW1-Pad7)
- SW1 pad 8: Net-(J4-Pad10) -> Net-(SW1-Pad8)
- U4 pad 40: Net-(J4-Pad8) -> Net-(SW1-Pad1)
- U4 pad 41: Net-(J4-Pad6) -> Net-(SW1-Pad2)
- U4 pad 42: Net-(J4-Pad5) -> Net-(SW1-Pad3)
- U4 pad 43: Net-(J4-Pad7) -> Net-(SW1-Pad4)
- U4 pad 44: Net-(J4-Pad9) -> Net-(SW1-Pad5)
- U4 pad 45: Net-(J4-Pad11) -> Net-(SW1-Pad6)
- U4 pad 46: Net-(J4-Pad12) -> Net-(SW1-Pad7)
- U4 pad 47: Net-(J4-Pad10) -> Net-(SW1-Pad8)
Routing:
- net Net-(SW1-Pad8): track 0.00 -> 148.1 mm
- net Net-(J4-Pad10): track 140.4 -> 0.00 mm
- net Net-(SW1-Pad7): track 0.00 -> 138.8 mm
- net Net-(J4-Pad12): track 129.7 -> 0.00 mm
- net Net-(J4-Pad11): track 121.0 -> 0.00 mm
- net Net-(SW1-Pad6): track 0.00 -> 119.1 mm
- net Net-(J4-Pad9): track 117.0 -> 0.00 mm
- net Net-(J4-Pad8): track 116.7 -> 0.00 mm
- net Net-(SW1-Pad5): track 0.00 -> 115.1 mm
- net Net-(J4-Pad6): track 114.7 -> 0.00 mm
- net Net-(J4-Pad7): track 112.0 -> 0.00 mm
- net Net-(SW1-Pad4): track 0.00 -> 111.1 mm
- net Net-(SW1-Pad1): track 0.00 -> 109.2 mm
- net Net-(J4-Pad5): track 107.6 -> 0.00 mm
- net Net-(SW1-Pad3): track 0.00 -> 107.4 mm
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